File: DRF1268T.kicad_pcb (KiCad board)
At the start: 2 copper layers, 5 parts, among them J1 SMA-J-P-X-RA-TH1, J2 Conn_01x08

Commit message: afasdf
Parts:
- added J3: Conn_01x01_Male, Connector_PinHeader_2.54mm:PinHeader_1x01_P2.54mm_Vertical, F.Cu at (127.5, 114.6)
- added J4: Conn_01x01_Male, Connector_PinHeader_2.54mm:PinHeader_1x01_P2.54mm_Vertical, F.Cu at (122.9, 114.6)
- J2: footprint Connector_PinSocket_2.54mm:PinSocket_1x08_P2.54mm_Vertical -> Connector_PinHeader_2.54mm:PinHeader_1x08_P2.54mm_Vertical
- moved J2 1.34 mm to (158.2, 92.0)

Commit message: First draft
Parts:
- removed J4: Conn_01x01_Male, Connector_PinHeader_2.54mm:PinHeader_1x01_P2.54mm_Vertical
- added REF**: MountingHole_2.2mm_M2, MountingHole:MountingHole_2.2mm_M2, F.Cu at (162.3, 71.9)
- added REF**: MountingHole_2.2mm_M2, MountingHole:MountingHole_2.2mm_M2, F.Cu at (141.2, 71.9)
- added REF**: MountingHole_2.2mm_M2, MountingHole:MountingHole_2.2mm_M2, F.Cu at (162.3, 101.6)
- added REF**: MountingHole_2.2mm_M2, MountingHole:MountingHole_2.2mm_M2, F.Cu at (141.2, 101.6)
- J3: value Conn_01x01_Male -> Conn_01x02_Male; footprint Connector_PinHeader_2.54mm:PinHeader_1x01_P2.54mm_Vertical -> Connector_PinHeader_2.54mm:PinHeader_1x02_P2.54mm_Vertical
- moved J1 32.8 mm to (156.1, 77.7)
- moved C1 32.3 mm to (142.2, 84.8)
- moved C2 28.4 mm to (142.3, 86.9)
- moved J3 25.9 mm to (142.2, 93.2)
- moved J2 14.6 mm to (162.6, 78.0)
- moved R1 12.0 mm to (145.4, 98.9)
Connections:
- J3 pad 1: GND -> +3.3V
Routing:
- net GND: track 0.00 -> 47.5 mm
- net +3.3V: track 0.00 -> 23.1 mm
- net Net-(J1-Pad1): track 0.00 -> 15.7 mm, vias 0 -> 1
- net Net-(R1-Pad16): track 0.00 -> 8.43 mm
- net Net-(R1-Pad15): track 0.00 -> 7.69 mm
- net Net-(R1-Pad14): track 0.00 -> 6.95 mm
- net Net-(R1-Pad13): track 0.00 -> 6.21 mm
- net Net-(R1-Pad12): track 0.00 -> 5.53 mm
- net Net-(R1-Pad11): track 0.00 -> 5.22 mm
- net Net-(R1-Pad10): track 0.00 -> 4.91 mm
- net Net-(R1-Pad9): track 0.00 -> 4.61 mm
Other:
- board outline added: 26.2 x 34.8 mm

Commit message: Changes to pcb layout
Parts:
- removed REF** (x4): MountingHole_2.2mm_M2, MountingHole:MountingHole_2.2mm_M2
- C1, C2: footprint Capacitor_SMD:C_0201_0603Metric -> Capacitor_SMD:C_0201_0603Metric_Pad0.64x0.40mm_HandSolder
- moved J1 4.50 mm to (151.6, 78.5), turned to -90 degrees
- moved J2 2.08 mm to (161.3, 79.6)
- moved J3 1.62 mm to (142.2, 94.8)
- moved C2 1.20 mm to (142.2, 88.1), turned to 90 degrees
- moved R1 0.63 mm to (144.7, 98.9)
- turned C1 to 90 degrees
Connections:
- J3 pad 1: +3.3V -> GND
- J3 pad 2: GND -> +3.3V
Routing:
- net GND: track 47.5 -> 0.00 mm
- net Net-(J1-Pad1): track 15.7 -> 11.2 mm, vias 1 -> 0
- net Net-(J2-Pad7): track 4.91 -> 3.60 mm
- net Net-(J2-Pad8): track 4.61 -> 3.31 mm
- net Net-(J2-Pad6): track 5.22 -> 3.97 mm
- net Net-(J2-Pad1): track 8.43 -> 7.44 mm
- net Net-(J2-Pad2): track 7.69 -> 6.83 mm
- net Net-(J2-Pad5): track 5.53 -> 4.72 mm
- net Net-(J2-Pad3): track 6.95 -> 6.38 mm
- net Net-(J2-Pad4): track 6.21 -> 5.71 mm
- added copper zone on B.Cu, net +3.3V
- added copper zone on F.Cu, net GND
Other:
- board size 26.2 x 34.8 mm -> 23.6 x 25.4 mm

Commit message: Changed
Parts:
- removed J3: Conn_01x02_Male, Connector_PinHeader_2.54mm:PinHeader_1x02_P2.54mm_Vertical
- C2: value C -> 10uF
- J2: value Conn_01x08 -> Conn_01x10_Male; footprint Connector_PinHeader_2.54mm:PinHeader_1x08_P2.54mm_Vertical -> Connector_PinSocket_2.54mm:PinSocket_1x10_P2.54mm_Vertical
- moved C1 27.8 mm to (165.9, 99.3)
- moved C2 26.5 mm to (164.4, 102.6)
- moved R1 23.8 mm to (152.4, 121.5)
- moved J1 23.6 mm to (159.3, 100.8)
- moved J2 18.9 mm to (168.7, 97.1)
Connections:
- J2 pad 1: Net-(J2-Pad1) -> +3.3V
- J2 pad 2: Net-(J2-Pad2) -> GND
- J2 pad 3: Net-(J2-Pad3) -> Net-(R1-Pad16)
- J2 pad 4: Net-(J2-Pad4) -> Net-(R1-Pad15)
- J2 pad 5: Net-(J2-Pad5) -> Net-(R1-Pad14)
- J2 pad 6: Net-(J2-Pad6) -> Net-(R1-Pad13)
- J2 pad 7: Net-(J2-Pad7) -> Net-(R1-Pad12)
- J2 pad 8: Net-(J2-Pad8) -> Net-(R1-Pad11)
- R1 pad 10: Net-(J2-Pad7) -> Net-(R1-Pad10)
- R1 pad 11: Net-(J2-Pad6) -> Net-(R1-Pad11)
- R1 pad 12: Net-(J2-Pad5) -> Net-(R1-Pad12)
- R1 pad 13: Net-(J2-Pad4) -> Net-(R1-Pad13)
- R1 pad 14: Net-(J2-Pad3) -> Net-(R1-Pad14)
- R1 pad 15: Net-(J2-Pad2) -> Net-(R1-Pad15)
- R1 pad 16: Net-(J2-Pad1) -> Net-(R1-Pad16)
- R1 pad 9: Net-(J2-Pad8) -> Net-(R1-Pad9)
Routing:
- net +3.3V: track 22.7 -> 5.17 mm, vias 0 -> 4
- net Net-(J2-Pad1): track 7.44 -> 0.00 mm
- net Net-(J2-Pad2): track 6.83 -> 0.00 mm
- net Net-(R1-Pad16): track 0.00 -> 6.44 mm
- net Net-(J2-Pad3): track 6.38 -> 0.00 mm
- net Net-(J2-Pad4): track 5.71 -> 0.00 mm
- net Net-(R1-Pad15): track 0.00 -> 5.70 mm
- net Net-(R1-Pad14): track 0.00 -> 4.96 mm
- net Net-(J2-Pad5): track 4.72 -> 0.00 mm
- net Net-(R1-Pad13): track 0.00 -> 4.27 mm
- net Net-(J2-Pad6): track 3.97 -> 0.00 mm
- net Net-(R1-Pad12): track 0.00 -> 3.97 mm
- net Net-(R1-Pad11): track 0.00 -> 3.66 mm
- net Net-(J2-Pad7): track 3.60 -> 0.00 mm
- net Net-(R1-Pad10): track 0.00 -> 3.35 mm
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Other:
- board size 23.6 x 25.4 mm -> 19.6 x 27.4 mm
- board text added: "ES"

Commit message: edits
Parts:
- moved C1 19.1 mm to (168.1, 118.2)
- moved J1 13.6 mm to (147.3, 107.3), turned to 90 degrees
- moved C2 7.80 mm to (168.3, 109.4)
- moved J2 1.49 mm to (167.9, 98.3), turned to -90 degrees
Routing:
- net Net-(R1-Pad9): track 3.05 -> 34.2 mm
- net Net-(R1-Pad10): track 3.35 -> 30.8 mm
- net Net-(R1-Pad11): track 3.66 -> 26.3 mm
- net Net-(R1-Pad12): track 3.97 -> 24.1 mm
- net Net-(R1-Pad13): track 4.27 -> 18.1 mm
- net Net-(R1-Pad14): track 4.96 -> 16.0 mm
- net Net-(R1-Pad15): track 5.70 -> 13.8 mm
- net Net-(J1-Pad1): track 11.2 -> 5.78 mm
- net Net-(R1-Pad16): track 6.44 -> 9.02 mm
- net GND: vias 0 -> 6
Other:
- board size 19.6 x 27.4 mm -> 27.4 x 25.7 mm
- board text added: "3.3V"
- board text added: "BUSY"
- board text added: "DIO1"
- board text added: "DIO2"
- board text added: "DRF1628T"
- board text added: "GND"
- board text added: "MISO"
- board text added: "MOSI"
- board text added: "NSS"
- board text added: "RST"
- board text added: "SCK"

Commit message: Changes
Routing:
- net GND: track 0.00 -> 5.73 mm, vias 6 -> 8
- net Net-(R1-Pad9): track 34.2 -> 35.3 mm
- net Net-(R1-Pad16): track 9.02 -> 10.2 mm
- net Net-(R1-Pad15): track 13.8 -> 14.9 mm
- net Net-(R1-Pad14): track 16.0 -> 17.1 mm
- net Net-(R1-Pad13): track 18.1 -> 19.3 mm
- net Net-(R1-Pad12): track 24.1 -> 25.2 mm
- net Net-(R1-Pad10): track 30.8 -> 32.0 mm
- net Net-(R1-Pad11): track 26.3 -> 27.4 mm
Changed lines of the file:
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@@
       (outputformat 1)
       (mirror false)
-      (drillshape 1)
+      (drillshape 0)
       (scaleselection 1)
-      (outputdirectory "")
+      (outputdirectory "/Users/ezzatsuhaime/Documents/DRF1268T/fab_files/")
     )
   )
@@
   (via (at 168.275 110.918) (size 0.8) (drill 0.4) (layers "F.Cu" "B.Cu") (net 1))
   (segment (start 153.098 107.318) (end 147.32 107.318) (width 0.2) (layer "F.Cu") (net 3))
+  (segment (start 145.542 106.553) (end 145.669 106.553) (width 0.2) (layer "F.Cu") (net 4))
+  (segment (start 148.082 109.093) (end 149.098 108.077) (width 0.2) (layer "F.Cu") (net 4))
+  (segment (start 146.558 105.664) (end 148.082 105.664) (width 0.2) (layer "F.Cu") (net 4))
+  (segment (start 148.209 105.664) (end 149.098 106.553) (width 0.2) (layer "F.Cu") (net 4))
+  (segment (start 145.669 106.553) (end 146.558 105.664) (width 0.2) (layer "F.Cu") (net 4))
+  (segment (start 148.082 105.664) (end 148.209 105.664) (width 0.2) (layer "F.Cu") (net 4))
+  (via (at 149.098 106.553) (size 0.4) (drill 0.2) (layers "F.Cu" "B.Cu") (free) (net 4))
   (via (at 145.542 106.553) (size 0.4) (drill 0.2) (layers "F.Cu" "B.Cu") (free) (net 4))
   (via (at 148.082 105.664) (size 0.4) (drill 0.2) (layers "F.Cu" "B.Cu") (free) (net 4))
@@
   (via (at 146.558 105.664) (size 0.4) (drill 0.2) (layers "F.Cu" "B.Cu") (free) (net 4))
   (via (at 146.558 109.093) (size 0.4) (drill 0.2) (layers "F.Cu" "B.Cu") (free) (net 4))
+  (via (at 149.098 108.077) (size 0.4) (drill 0.2) (layers "F.Cu" "B.Cu") (free) (net 4))
   (via (at 145.542 108.077) (size 0.4) (drill 0.2) (layers "F.Cu" "B.Cu") (free) (net 4))
-  (segment (start 156.337 113.411) (end 162.844 119.918) (width 0.25) (layer "F.Cu") (net 5))
-  (segment (start 145.004 101.697) (end 146.304 102.997) (width 0.25) (layer "F.Cu") (net 5))
-  (segment (start 156.337 106.939584) (end 156.337 113.411) (width 0.25) (layer "F.Cu") (net 5))
-  (segment (start 162.844 119.918) (end 165.608 119.918) (width 0.25) (layer "F.Cu") (net 5))
-  (segment (start 145.004 101.697) (end 145.004 99.466) (width 0.25) (layer "F.Cu") (net 5))
-  (segment (start 152.394416 102.997) (end 156.337 106.939584) (width 0.25) (layer "F.Cu") (net 5))
-  (segment (start 146.304 102.997) (end 152.394416 102.997) (width 0.25) (layer "F.Cu") (net 5))
-  (segment (start 148.521 102.547) (end 152.580812 102.547) (width 0.25) (layer "F.Cu") (net 6))
-  (segment (start 147.544 101.57) (end 147.544 99.466) (width 0.25) (layer "F.Cu") (net 6))
-  (segment (start 156.787 113.224604) (end 161.680396 118.118) (width 0.25) (layer "F.Cu") (net 6))
-  (segment (start 156.787 106.753188) (end 156.787 113.224604) (width 0.25) (layer "F.Cu") (net 6))
-  (segment (start 147.544 101.57) (end 148.521 102.547) (width 0.25) (layer "F.Cu") (net 6))
-  (segment (start 152.580812 102.547) (end 156.787 106.753188) (width 0.25) (layer "F.Cu") (net 6))
-  (segment (start 161.680396 118.118) (end 165.608 118.118) (width 0.25) (layer "F.Cu") (net 6))
+  (segment (start 152.394416 102.997) (end 146.304 102.997) (width 0.25) (layer "F.Cu") (net 5))
+  (segment (start 165.608 119.918) (end 162.844 119.918) (width 0.25) (layer "F.Cu") (net 5))
+  (segment (start 162.844 119.918) (end 156.337 113.411) (width 0.25) (layer "F.Cu") (net 5))
+  (segment (start 146.304 102.997) (end 145.004 101.697) (width 0.25) (layer "F.Cu") (net 5))
+  (segment (start 156.337 106.939584) (end 152.394416 102.997) (width 0.25) (layer "F.Cu") (net 5))
+  (segment (start 156.337 113.411) (end 156.337 106.939584) (width 0.25) (layer "F.Cu") (net 5))
+  (segment (start 145.004 101.697) (end 145.004 98.323) (width 0.25) (layer "F.Cu") (net 5))
+  (segment (start 147.544 101.57) (end 147.544 98.323) (width 0.25) (layer "F.Cu") (net 6))
+  (segment (start 161.680396 118.118) (end 156.787 113.224604) (width 0.25) (layer "F.Cu") (net 6))
+  (segment (start 152.580812 102.547) (end 148.521 102.547) (width 0.25) (layer "F.Cu") (net 6))
+  (segment (start 156.787 113.224604) (end 156.787 106.753188) (width 0.25) (layer "F.Cu") (net 6))
+  (segment (start 148.521 102.547) (end 147.544 101.57) (width 0.25) (layer "F.Cu") (net 6))
+  (segment (start 165.608 118.118) (end 161.680396 118.118) (width 0.25) (layer "F.Cu") (net 6))
+  (segment (start 156.787 106.753188) (end 152.580812 102.547) (width 0.25) (layer "F.Cu") (net 6))
+  (segment (start 150.084 99.413792) (end 150.084 98.323) (width 0.25) (layer "F.Cu") (net 7))
   (segment (start 165.608 116.318) (end 160.516792 116.318) (width 0.25) (layer "F.Cu") (net 7))
   (segment (start 157.295 106.624792) (end 150.084 99.413792) (width 0.25) (layer "F.Cu") (net 7))
   (segment (start 160.516792 116.318) (end 157.295 113.096208) (width 0.25) (layer "F.Cu") (net 7))
   (segment (start 157.295 113.096208) (end 157.295 106.624792) (width 0.25) (layer "F.Cu") (net 7))
+  (segment (start 159.353188 114.518) (end 157.745 112.909812) (width 0.25) (layer "F.Cu") (net 8))
   (segment (start 165.608 114.518) (end 159.353188 114.518) (width 0.25) (layer "F.Cu") (net 8))
-  (segment (start 159.353188 114.518) (end 157.745 112.909812) (width 0.25) (layer "F.Cu") (net 8))
-  (segment (start 152.624 101.317396) (end 152.624 99.466) (width 0.25) (layer "F.Cu") (net 8))
+  (segment (start 152.624 101.317396) (end 152.624 98.323) (width 0.25) (layer "F.Cu") (net 8))
   (segment (start 157.745 106.438396) (end 152.624 101.317396) (width 0.25) (layer "F.Cu") (net 8))
   (segment (start 157.745 112.909812) (end 157.745 106.438396) (width 0.25) (layer "F.Cu") (net 8))
   (segment (start 165.608 112.718) (end 164.661 112.718) (width 0.25) (layer "F.Cu") (net 9))
   (segment (start 164.661 112.718) (end 155.164 103.221) (width 0.25) (layer "F.Cu") (net 9))
-  (segment (start 155.164 103.221) (end 155.164 99.466) (width 0.25) (layer "F.Cu") (net 9))
-  (segment (start 157.704 105.124604) (end 157.704 99.466) (width 0.25) (layer "F.Cu") (net 10))
+  (segment (start 155.164 103.221) (end 155.164 98.323) (width 0.25) (layer "F.Cu") (net 9))
+  (segment (start 163.497396 110.918) (end 157.704 105.124604) (width 0.25) (layer "F.Cu") (net 10))
+  (segment (start 157.704 105.124604) (end 157.704 98.323) (width 0.25) (layer "F.Cu") (net 10))
   (segment (start 165.608 110.918) (end 163.497396 110.918) (width 0.25) (layer "F.Cu") (net 10))
-  (segment (start 163.497396 110.918) (end 157.704 105.124604) (width 0.25) (layer "F.Cu") (net 10))
   (segment (start 165.608 109.118) (end 162.333792 109.118) (width 0.25) (layer "F.Cu") (net 11))
-  (segment (start 160.244 107.028208) (end 160.244 99.466) (width 0.25) (layer "F.Cu") (net 11))
   (segment (start 162.333792 109.118) (end 160.244 107.028208) (width 0.25) (layer "F.Cu") (net 11))
-  (segment (start 162.784 104.494) (end 165.608 107.318) (width 0.25) (layer "F.Cu") (net 12))
-  (segment (start 162.784 104.494) (end 162.784 99.466) (width 0.25) (layer "F.Cu") (net 12))
+  (segment (start 160.244 107.028208) (end 160.244 98.323) (width 0.25) (layer "F.Cu") (net 11))
+  (segment (start 162.784 104.494) (end 162.784 98.323) (width 0.25) (layer "F.Cu") (net 12))
+  (segment (start 165.608 107.318) (end 162.784 104.494) (width 0.25) (layer "F.Cu") (net 12))
   (zone (net 4) (net_name "GND") (layer "F.Cu") (hatch edge 0.508)
     (connect_pads (clearance 0.508))
